Commit message: datasets test

File: legged_gym/resources/robots/adam_sp/adam_sp_yrr.urdf (robot description, URDF)
Before this commit: robot adam_sp, 77 links, 76 joints
Links:
- removed link keyframe_head_link
- removed link keyframe_left_ankle_link
- removed link keyframe_left_collar_link
- removed link keyframe_left_elbow_link
- removed link keyframe_left_hip_link
- removed link keyframe_left_knee_link
- removed link keyframe_left_shoulder_link
- removed link keyframe_left_wrist_link
- removed link keyframe_pelvis_link
- removed link keyframe_right_ankle_link
- removed link keyframe_right_collar_link
- removed link keyframe_right_elbow_link
- removed link keyframe_right_hip_link
- removed link keyframe_right_knee_link
- removed link keyframe_right_shoulder_link
- removed link keyframe_right_wrist_link
- removed link keyframe_torso_link
- removed link left_ankle_roll_side1
- removed link left_ankle_roll_side2
- removed link mid360_link
- removed link right_ankle_roll_side1
- removed link right_ankle_roll_side2
- link L_index_distal: geometry visual mesh filename=../meshes_stl_0.25/L_index_distal.STL
- link L_index_proximal: geometry visual mesh filename=../meshes_stl_0.25/L_index_proximal.STL
- link L_middle_distal: geometry visual mesh filename=../meshes_stl_0.25/L_middle_distal.STL
- link L_middle_proximal: geometry visual mesh filename=../meshes_stl_0.25/L_middle_proximal.STL
- link L_pinky_distal: geometry visual mesh filename=../meshes_stl_0.25/L_pinky_distal.STL
- link L_pinky_proximal: geometry visual mesh filename=../meshes_stl_0.25/L_pinky_proximal.STL
- link L_ring_distal: geometry visual mesh filename=../meshes_stl_0.25/L_ring_distal.STL
- link L_ring_proximal: geometry visual mesh filename=../meshes_stl_0.25/L_ring_proximal.STL
- link L_thumb_distal: geometry visual mesh filename=../meshes_stl_0.25/L_thumb_distal.STL
- link L_thumb_intermediate: geometry visual mesh filename=../meshes_stl_0.25/L_thumb_intermediate.STL
- link L_thumb_proximal: geometry visual mesh filename=../meshes_stl_0.25/L_thumb_proximal.STL
- link L_thumb_proximal_base: geometry visual mesh filename=../meshes_stl_0.25/L_thumb_proximal_base.STL
- link R_index_distal: geometry visual mesh filename=../meshes_stl_0.25/R_index_distal.STL
- link R_index_proximal: geometry visual mesh filename=../meshes_stl_0.25/R_index_proximal.STL
- link R_middle_distal: geometry visual mesh filename=../meshes_stl_0.25/R_middle_distal.STL
- link R_middle_proximal: geometry visual mesh filename=../meshes_stl_0.25/R_middle_proximal.STL
- link R_pinky_distal: geometry visual mesh filename=../meshes_stl_0.25/R_pinky_distal.STL
- link R_pinky_proximal: geometry visual mesh filename=../meshes_stl_0.25/R_pinky_proximal.STL
- link R_ring_distal: geometry visual mesh filename=../meshes_stl_0.25/R_ring_distal.STL
- link R_ring_proximal: geometry visual mesh filename=../meshes_stl_0.25/R_ring_proximal.STL
- link R_thumb_distal: geometry visual mesh filename=../meshes_stl_0.25/R_thumb_distal.STL
- link R_thumb_intermediate: geometry visual mesh filename=../meshes_stl_0.25/R_thumb_intermediate.STL
- link R_thumb_proximal: geometry visual mesh filename=../meshes_stl_0.25/R_thumb_proximal.STL
- link R_thumb_proximal_base: geometry visual mesh filename=../meshes_stl_0.25/R_thumb_proximal_base.STL
- link anklePitchLeft: geometry visual mesh filename=../meshes_stl_0.25/anklePitchLeft.STL
- link anklePitchRight: geometry visual mesh filename=../meshes_stl_0.25/anklePitchRight.STL
- link elbowLeft: geometry visual mesh filename=../meshes_stl_0.25/elbowLeft.STL
- link elbowRight: geometry visual mesh filename=../meshes_stl_0.25/elbowRight.STL
- link hipPitchLeft: geometry visual mesh filename=../meshes_stl_0.25/hipPitchLeft.STL
- link hipPitchRight: geometry visual mesh filename=../meshes_stl_0.25/hipPitchRight.STL
- link hipRollLeft: geometry visual mesh filename=../meshes_stl_0.25/hipRollLeft.STL
- link hipRollRight: geometry visual mesh filename=../meshes_stl_0.25/hipRollRight.STL
- link pelvis: geometry collision cylinder length=0.2 radius=0.1; visual mesh filename=../meshes_stl_0.25/pelvis.STL
- link shinLeft: geometry collision box size=0.08 0.06 0.2; visual mesh filename=../meshes_stl_0.25/shinLeft.STL
- link shinRight: geometry collision box size=0.08 0.06 0.2; visual mesh filename=../meshes_stl_0.25/shinRight.STL
- link shoulderPitchLeft: geometry visual mesh filename=../meshes_stl_0.25/shoulderPitchLeft.STL
- link shoulderPitchRight: geometry visual mesh filename=../meshes_stl_0.25/shoulderPitchRight.STL
- link shoulderRollLeft: geometry visual mesh filename=../meshes_stl_0.25/shoulderRollLeft.STL
- link shoulderRollRight: geometry visual mesh filename=../meshes_stl_0.25/shoulderRollRight.STL
- link shoulderYawLeft: geometry collision cylinder length=0.15 radius=0.038; visual mesh filename=../meshes_stl_0.25/shoulderYawLeft.STL
- link shoulderYawRight: geometry collision cylinder length=0.15 radius=0.038; visual mesh filename=../meshes_stl_0.25/shoulderYawRight.STL
- link thighLeft: geometry collision mesh filename=../meshes_stl_0.25/thighLeft.STL; visual mesh filename=../meshes_stl_0.25/thighLeft.STL
- link thighRight: geometry collision mesh filename=../meshes_stl_0.25/thighRight.STL; visual mesh filename=../meshes_stl_0.25/thighRight.STL
- link toeLeft: geometry collision box size=0.24 0.1 0.02; visual mesh filename=../meshes_stl_0.25/toeLeft.STL
- link toeRight: geometry collision box size=0.24 0.1 0.02; visual mesh filename=../meshes_stl_0.25/toeRight.STL
- link torso: geometry collision sphere radius=0.13; visual mesh filename=../meshes_stl_0.25/torso.STL
- link waistPitch_link: geometry visual mesh filename=../meshes_stl_0.25/waistPitch_link.STL
- link waistRoll_link: geometry visual mesh filename=../meshes_stl_0.25/waistRoll_link.STL
- link wristPitchLeft: geometry visual mesh filename=../meshes_stl_0.25/wristPitchLeft.STL
- link wristPitchRight: geometry visual mesh filename=../meshes_stl_0.25/wristPitchRight.STL
- link wristRollLeft: geometry visual mesh filename=../meshes_stl_0.25/wristRollLeft.STL
- link wristRollRight: geometry visual mesh filename=../meshes_stl_0.25/wristRollRight.STL
- link wristYawLeft: geometry collision mesh filename=../meshes_stl_0.25/wristYawLeft.STL; visual mesh filename=../meshes_stl_0.25/wristYawLeft.STL
- link wristYawRight: geometry collision mesh filename=../meshes_stl_0.25/wristYawRight.STL; visual mesh filename=../meshes_stl_0.25/wristYawRight.STL
Joints:
- removed joint auxiliary_left_ankle_roll_joint4
- removed joint auxiliary_right_ankle_roll_joint3
- removed joint keyframe_head_joint
- removed joint keyframe_left_ankle_joint
- removed joint keyframe_left_collar_joint
- removed joint keyframe_left_elbow_joint
- removed joint keyframe_left_hip_joint
- removed joint keyframe_left_knee_joint
- removed joint keyframe_left_shoulder_joint
- removed joint keyframe_left_wrist_joint
- removed joint keyframe_pelvis_joint
- removed joint keyframe_right_ankle_joint
- removed joint keyframe_right_collar_joint
- removed joint keyframe_right_elbow_joint
- removed joint keyframe_right_hip_joint
- removed joint keyframe_right_knee_joint
- removed joint keyframe_right_shoulder_joint
- removed joint keyframe_right_wrist_joint
- removed joint keyframe_torso_joint
- removed joint left_ankle_roll_side1
- removed joint mid360_joint
- removed joint right_ankle_roll_side2
- joint wristPitch_Left: type revolute -> fixed
- joint wristPitch_Right: type revolute -> fixed
- joint wristRoll_Left: type revolute -> fixed
- joint wristRoll_Right: type revolute -> fixed
- joint wristYaw_Left: type revolute -> fixed
- joint wristYaw_Right: type revolute -> fixed
