Commit message: fix collision

File: legged_gym/resources/robots/adam_sp/adam_sp.urdf (robot description, URDF)
Before this commit: robot adam_sp, 73 links, 72 joints
Links:
- link L_index_distal: geometry visual mesh filename=meshes_stl_0.25/L_index_distal.STL
- link L_index_proximal: geometry visual mesh filename=meshes_stl_0.25/L_index_proximal.STL
- link L_middle_distal: geometry visual mesh filename=meshes_stl_0.25/L_middle_distal.STL
- link L_middle_proximal: geometry visual mesh filename=meshes_stl_0.25/L_middle_proximal.STL
- link L_pinky_distal: geometry visual mesh filename=meshes_stl_0.25/L_pinky_distal.STL
- link L_pinky_proximal: geometry visual mesh filename=meshes_stl_0.25/L_pinky_proximal.STL
- link L_ring_distal: geometry visual mesh filename=meshes_stl_0.25/L_ring_distal.STL
- link L_ring_proximal: geometry visual mesh filename=meshes_stl_0.25/L_ring_proximal.STL
- link L_thumb_distal: geometry visual mesh filename=meshes_stl_0.25/L_thumb_distal.STL
- link L_thumb_proximal: geometry visual mesh filename=meshes_stl_0.25/L_thumb_proximal.STL
- link L_thumb_proximal_base: geometry visual mesh filename=meshes_stl_0.25/L_thumb_proximal_base.STL
- link R_index_distal: geometry visual mesh filename=meshes_stl_0.25/R_index_distal.STL
- link R_index_proximal: geometry visual mesh filename=meshes_stl_0.25/R_index_proximal.STL
- link R_middle_distal: geometry visual mesh filename=meshes_stl_0.25/R_middle_distal.STL
- link R_middle_proximal: geometry visual mesh filename=meshes_stl_0.25/R_middle_proximal.STL
- link R_pinky_distal: geometry visual mesh filename=meshes_stl_0.25/R_pinky_distal.STL
- link R_pinky_proximal: geometry visual mesh filename=meshes_stl_0.25/R_pinky_proximal.STL
- link R_ring_distal: geometry visual mesh filename=meshes_stl_0.25/R_ring_distal.STL
- link R_ring_proximal: geometry visual mesh filename=meshes_stl_0.25/R_ring_proximal.STL
- link R_thumb_distal: geometry visual mesh filename=meshes_stl_0.25/R_thumb_distal.STL
- link R_thumb_proximal: geometry visual mesh filename=meshes_stl_0.25/R_thumb_proximal.STL
- link R_thumb_proximal_base: geometry visual mesh filename=meshes_stl_0.25/R_thumb_proximal_base.STL
- link anklePitchLeft: geometry visual mesh filename=meshes_stl_0.25/anklePitchLeft.STL
- link anklePitchRight: geometry visual mesh filename=meshes_stl_0.25/anklePitchRight.STL
- link elbowLeft: geometry visual mesh filename=meshes_stl_0.25/elbowLeft.STL
- link elbowRight: geometry visual mesh filename=meshes_stl_0.25/elbowRight.STL
- link hipRollLeft: geometry visual mesh filename=meshes_stl_0.25/hipRollLeft.STL
- link hipRollRight: geometry visual mesh filename=meshes_stl_0.25/hipRollRight.STL
- link pelvis: geometry collision cylinder length=0.2 radius=0.1; visual mesh filename=meshes_stl_0.25/pelvis.STL
- link shinLeft: geometry collision box size=0.08 0.06 0.2; visual mesh filename=meshes_stl_0.25/shinLeft.STL
- link shinRight: geometry collision box size=0.08 0.06 0.2; visual mesh filename=meshes_stl_0.25/shinRight.STL
- link shoulderPitchLeft: geometry visual mesh filename=meshes_stl_0.25/shoulderPitchLeft.STL
- link shoulderPitchRight: geometry visual mesh filename=meshes_stl_0.25/shoulderPitchRight.STL
- link shoulderRollLeft: geometry visual mesh filename=meshes_stl_0.25/shoulderRollLeft.STL
- link shoulderRollRight: geometry visual mesh filename=meshes_stl_0.25/shoulderRollRight.STL
- link shoulderYawLeft: geometry collision cylinder length=0.15 radius=0.038; visual mesh filename=meshes_stl_0.25/shoulderYawLeft.STL
- link shoulderYawRight: geometry collision cylinder length=0.15 radius=0.038; visual mesh filename=meshes_stl_0.25/shoulderYawRight.STL
- link torso: geometry collision sphere radius=0.13; visual mesh filename=meshes_stl_0.25/torso.STL
- link waistPitch_link: geometry visual mesh filename=meshes_stl_0.25/waistPitch_link.STL
- link wristPitchLeft: geometry visual mesh filename=meshes_stl_0.25/wristPitchLeft.STL
- link wristPitchRight: geometry visual mesh filename=meshes_stl_0.25/wristPitchRight.STL

Commit message: tmp save, ready test

File: legged_gym/resources/robots/adam_sp/adam_sp.urdf (robot description, URDF)
Before this commit: robot adam_sp, 77 links, 76 joints
Joints:
- joint keyframe_head_joint: origin xyz=0 0 0 rpy=0 0 0 -> xyz=0 0 0.4 rpy=0 0 0
- joint keyframe_left_ankle_joint: origin xyz=0 0 0 rpy=0 0 0 -> xyz=0.0 0.0 -0.061 rpy=0 0 0
- joint keyframe_left_collar_joint: origin xyz=0 0 0 rpy=0 0 0 -> xyz=0 0 0.0 rpy=0 0 0
- joint keyframe_left_hip_joint: parent hipPitchLeft -> hipRollLeft
- joint keyframe_left_shoulder_joint: parent shoulderPitchLeft -> shoulderRollLeft
- joint keyframe_right_ankle_joint: origin xyz=0 0 0 rpy=0 0 0 -> xyz=0.0 0 -0.061 rpy=0 0 0
- joint keyframe_right_hip_joint: parent hipPitchRight -> hipRollRight
- joint keyframe_right_shoulder_joint: parent shoulderPitchRight -> shoulderRollRight
- joint keyframe_torso_joint: origin xyz=0 0 0 rpy=0 0 0 -> xyz=0 0 0.2 rpy=0 0 0

Commit message: fix ver

File: legged_gym/resources/robots/adam_sp/adam_sp.urdf (robot description, URDF)
Before this commit: robot adam_sp, 77 links, 76 joints
Joints:
- joint anklePitch_Left: limit lower=-1.0 upper=0.35 effort=40 velocity=20 -> lower=-1.0 upper=0.35 effort=80 velocity=20
- joint anklePitch_Right: limit lower=-1.0 upper=0.35 effort=40 velocity=20 -> lower=-1.0 upper=0.35 effort=80 velocity=20
- joint ankleRoll_Left: limit lower=-0.3491 upper=0.3491 effort=12 velocity=20 -> lower=-0.3491 upper=0.3491 effort=80 velocity=20
- joint ankleRoll_Right: limit lower=-0.3491 upper=0.3491 effort=12 velocity=20 -> lower=-0.3491 upper=0.3491 effort=80 velocity=20
- joint keyframe_pelvis_joint: origin xyz=0 0 0 rpy=0 0 0 -> xyz=0 0 -0.075 rpy=0 0 0
